File: minipowersupply.kicad_pcb (KiCad board)
At the start: 2 copper layers, 180 x 80 mm, 31 parts, among them J1 3.3V, J2 5V, J3 AdjustV, J4 Power In, SW1 SW_MEC_5G_LED, U1 AP64500SP-13

Commit message: increase size of pads, reorganize a bit
Parts:
- moved F3 16.9 mm to (234.7, 128.4)
- moved F2 16.9 mm to (176.7, 128.8)
- moved F1 16.8 mm to (118.7, 129.6)
Routing:
- net 3.3V: track 131.7 -> 108.3 mm
- net 5V: track 56.8 -> 39.9 mm
- net +VDC: track 79.6 -> 62.8 mm
- net Net-(J3-Pin_2): track 4.43 -> 19.5 mm
- net Net-(J2-Pin_2): track 4.56 -> 19.4 mm
- net Net-(J1-Pin_2): track 6.07 -> 18.4 mm
- net Net-(U2-Cout): track 2.91 -> 5.64 mm
- net Net-(U3-Cout): track 2.86 -> 4.84 mm
- net Net-(U4-Cout): track 3.06 -> 4.49 mm
- net Net-(U1-FB): track 35.7 -> 36.6 mm

Commit message: [pcb] misc
Parts:
- removed J4: Power In, Connector_PinSocket_2.54mm:PinSocket_2x07_P2.54mm_Vertical_SMD
- added C17: 10u, Capacitor_SMD:C_1206_3216Metric, B.Cu at (141.4, 86.7)
- added C20: 10u, Capacitor_SMD:C_0805_2012Metric, B.Cu at (148.6, 80.0)
- added J6: JST-PH2 Bat, Connector_JST:JST_PH_S9B-PH-SM4-TB_1x09-1MP_P2.00mm_Horizontal, B.Cu at (167.8, 82.6)
- added JP1: SolderJumper_2_Open, Jumper:SolderJumper-2_P1.3mm_Open_RoundedPad1.0x1.5mm, B.Cu at (142.6, 80.2)
- added U5: NCP1117-5_SOT223, Package_TO_SOT_SMD:SOT-223-3_TabPin2, B.Cu at (147.3, 86.4)
- H1, H2, H3, H4: footprint MountingHole:MountingHole_4.3mm_M4 -> MountingHole:MountingHole_4.3mm_M4_DIN965_Pad
- moved D2 13.7 mm to (182.2, 92.8), turned to 0 degrees
- moved D3 7.50 mm to (156.6, 87.4), turned to -90 degrees
- moved R3 4.85 mm to (204.6, 88.1)
- moved F3 4.06 mm to (238.3, 126.5)
- moved C5 2.50 mm to (206.9, 93.1)
- moved C6 2.29 mm to (202.0, 93.0)
- moved C7 2.29 mm to (204.6, 93.0)
- moved L1 1.68 mm to (195.4, 89.7)
- moved C2 0.52 mm to (184.2, 89.3)
Connections:
- C1 pad 2: GND -> Volt-GND
- C2 pad 2: GND -> Volt-GND
- C3 pad 2: GND -> Volt-GND
- C5 pad 2: GND -> Volt-GND
- C6 pad 2: GND -> Volt-GND
- C7 pad 2: GND -> Volt-GND
- D1 pad 2: GND -> Volt-GND
- D2 pad 2: GND -> Volt-GND
- D3 pad 2: GND -> Volt-GND
- F1 pad 1: Net-(U2-Cout) -> 3.3V
- F2 pad 1: Net-(U3-Cout) -> 5V
- F3 pad 1: Net-(U4-Cout) -> +VDC
- J1 pad 1: GND -> Net-(J1-Pin_1)
- J2 pad 1: GND -> Net-(J2-Pin_1)
- J3 pad 1: GND -> Net-(J3-Pin_1)
- R1 pad 2: GND -> Volt-GND
- R3 pad 2: GND -> Volt-GND
- SW1 pad 1: GND -> Volt-GND
- SW1 pad 2: GND -> Volt-GND
- U1 pad 7: GND -> Volt-GND
- U2 pad 1: GND -> Volt-GND
- U2 pad 2: 3.3V -> Volt-5V
- U2 pad 3: 3.3V -> Volt-GND
- U2 pad 4: Net-(U2-Cout) -> Net-(J1-Pin_1)
- U3 pad 1: GND -> Volt-GND
- U3 pad 2: 5V -> Volt-5V
- U3 pad 3: 5V -> Volt-GND
- U3 pad 4: Net-(U3-Cout) -> Net-(J2-Pin_1)
- U4 pad 1: GND -> Volt-GND
- U4 pad 2: +VDC -> Volt-5V
- U4 pad 3: +VDC -> Volt-GND
- U4 pad 4: Net-(U4-Cout) -> Net-(J3-Pin_1)
Routing:
- net Volt-5V: track 0.00 -> 251.6 mm
- net Net-(J1-Pin_1): track 0.00 -> 49.7 mm
- net Net-(J2-Pin_1): track 0.00 -> 49.6 mm
- net Net-(J3-Pin_1): track 0.00 -> 49.5 mm
- net 12V: track 21.8 -> 46.9 mm
- net 5V: track 39.9 -> 55.6 mm
- net +VDC: track 62.8 -> 78.3 mm
- net Volt-GND: track 0.00 -> 14.2 mm
- net Net-(U1-FB): track 36.6 -> 24.7 mm
- net Net-(J3-Pin_2): track 19.5 -> 31.0 mm
- net Net-(J1-Pin_2): track 18.4 -> 28.7 mm
- net Net-(J2-Pin_2): track 19.4 -> 28.6 mm
- net 3.3V: track 108.3 -> 116.5 mm
- net Power On: track 65.4 -> 71.9 mm
- net Net-(U2-Cout): track 5.64 -> 0.00 mm
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- added copper zone on B.Cu, net Volt-GND
- added copper zone on F.Cu, net Volt-GND
- removed copper zone on B.Cu, net GND
Other:
- board text added: "GND"
