File: minipowersupply.kicad_sch (KiCad schematic)
At the start: 32 parts, among them J1 3.3V, J2 5V, J3 AdjustV, J4 Power In, SW1 SW_MEC_5G_LED, U1 AP64500SP-13

Commit message: [pcb] misc
Parts:
- removed J4: Power In, Connector_PinSocket_2.54mm:PinSocket_2x07_P2.54mm_Vertical_SMD, symbol Connector_Generic:Conn_02x07_Odd_Even
- added C17: 10u, Capacitor_SMD:C_1206_3216Metric, symbol Device:C
- added C20: 10u, Capacitor_SMD:C_0805_2012Metric, symbol Device:C
- added J6: JST-PH2 Bat, Connector_JST:JST_PH_S9B-PH-SM4-TB_1x09-1MP_P2.00mm_Horizontal, symbol Connector_Generic:Conn_01x09
- added U5: NCP1117-5_SOT223, Package_TO_SOT_SMD:SOT-223-3_TabPin2, symbol Regulator_Linear:NCP1117-3.3_SOT223
- H1, H2, H3, H4: footprint MountingHole:MountingHole_4.3mm_M4 -> MountingHole:MountingHole_4.3mm_M4_DIN965_Pad; symbol Mechanical:MountingHole -> Mechanical:MountingHole_Pad; now left out of the parts list
Connections:
- net +VDC: now also F3.1; no longer U4.2 (Vin), U4.3 (Cin)
- net 12V: now also C20.1, J6.7 (Pin_7), J6.8 (Pin_8), U5.3 (VI)
- net 3.3V: now also F1.1, J6.3 (Pin_3), J6.4 (Pin_4); no longer U2.2 (Vin), U2.3 (Cin)
- net 5V: now also F2.1, J6.5 (Pin_5), J6.6 (Pin_6); no longer U3.2 (Vin), U3.3 (Cin)
- net GND: now also H1.1, H2.1, H3.1, H4.1, U2.3 (Cin), U3.3 (Cin), U4.3 (Cin), C17.2, C20.2, J6.1 (Pin_1), J6.2 (Pin_2), U5.1 (GND); no longer J1.1 (Pin_1), J2.1 (Pin_1), J3.1 (Pin_1)
- net Power On: now also J6.9 (Pin_9)
- net at U2.4 (Cout): now also J1.1 (Pin_1); no longer F1.1
- net at F1.2, J1.2 (Pin_2): now also U2.5 (Vprobe)
- net at U3.4 (Cout): now also J2.1 (Pin_1); no longer F2.1
- net at U4.4 (Cout): now also J3.1 (Pin_1); no longer F3.1
- net at F3.2, J3.2 (Pin_2): now also U4.5 (Vprobe)
- net at F2.2, J2.2 (Pin_2): now also U3.5 (Vprobe)
- new net Volt-5V: C17.1, U2.2 (Vin), U3.2 (Vin), U4.2 (Vin), U5.2 (VO)
Other:
- moved on the sheet: F1, F2, F3, J1, J2
